File: ADS1299_4_Feather.sch (EAGLE design)
At the start: 43 parts, among them U1 ADS1299-4PAG, U2 TPD4E1B06DRLR, U3 TPD4E1B06DRLR, U4 TPD4E1B06DRLR

Commit message: modified:   ADS1299_4_Feather.sch 	removed noise filters and changed component models
Parts:
- removed C20: 1nF, SparkFun-Capacitors:1000UF-RADIAL-5MM-25V-20%-NO-SILK
- removed U2, U3, U4: TPD4E1B06DRLR, TPD4E1B06DRLR:TPD4E1B06DRLR
- added C24: 1uF, SparkFun-Capacitors:10UF-POLAR-RADIAL-2.5MM-25V-20%
- C1, C2, C3, C4, C5, C9: device SparkFun-Capacitors:1000UF-RADIAL-5MM-25V-20%-NO-SILK -> SparkFun-Capacitors:10UF-POLAR-RADIAL-2.5MM-25V-20%
- C10: value 0.1uF -> 10uF; device SparkFun-Capacitors:1000UF-RADIAL-5MM-25V-20%-NO-SILK -> SparkFun-Capacitors:10UF-POLAR-RADIAL-2.5MM-25V-20%
- C11: value 1uF -> 0.1uF; device SparkFun-Capacitors:1000UF-RADIAL-5MM-25V-20%-NO-SILK -> SparkFun-Capacitors:10UF-POLAR-RADIAL-2.5MM-25V-20%
- C12, C13, C14, C15, C16, C17, C18, C19, C21, C22, C23: value 1nF -> 1 nF; device SparkFun-Capacitors:1000UF-RADIAL-5MM-25V-20%-NO-SILK -> adafruit:C-US025-024X044
- C6: value 10uF -> 1 nF; device SparkFun-Capacitors:1000UF-RADIAL-5MM-25V-20%-NO-SILK -> adafruit:C-US025-024X044
- C7: value 1uF -> 100uF; device SparkFun-Capacitors:1000UF-RADIAL-5MM-25V-20%-NO-SILK -> SparkFun-Capacitors:10UF-POLAR-RADIAL-2.5MM-25V-20%
- C8: value 100uF -> 1uF; device SparkFun-Capacitors:1000UF-RADIAL-5MM-25V-20%-NO-SILK -> SparkFun-Capacitors:10UF-POLAR-RADIAL-2.5MM-25V-20%
- JP1: value (none) -> 1x12
- JP2: value (none) -> 1x16
- JP3: value (none) -> 2x9
- R1, R10, R11, R12, R2, R3, R4, R5, R6, R7, R8: device adafruit:R-US_0207/10 -> SparkFun-Resistors:1MOHM-HORIZ-1/6W-5%
Connections:
- removed net 1N: JP3.14, R1.1, U2.IO1
- removed net 1P: JP3.13, R2.1, U2.IO2
- removed net 2N: JP3.12, R7.1, U3.IO3
- removed net 2P: JP3.11, R8.1, U3.IO4
- removed net 3N: JP3.10, R5.1, U3.IO1
- removed net 3P: JP3.9, R6.1, U3.IO2
- removed net 4N: JP3.8, R11.1, U4.IO3
- removed net 4P: JP3.7, R12.1, U4.IO4
- new net 1_N: JP3.14, R1.1
- new net 1_P: JP3.13, R2.1
- new net 2_N: JP3.12, R7.1
- new net 2_P: JP3.11, R8.1
- new net 3_N: JP3.10, R5.1
- new net 3_P: JP3.9, R6.1
- new net 4_N: JP3.8, R11.1
- new net 4_P: JP3.7, R10.1
- net 5V: no longer U4.IO1
- net BIAS: now also R12.1; no longer R10.1, U4.IO2
- net BIAS_DRV: now also C21.1, C6.1, R12.2; no longer C20.+, C22.+, R10.2
- net BIAS_IN: now also C6.2; no longer C20.-
- net GND: now also C12.2, C13.2, C14.2, C15.2, C16.2, C17.2, C18.2, C19.2, C21.2, C22.2, C23.2, C24.-, C5.-; no longer C10.-, C11.-, C12.-, C13.-, C14.-, C15.-, C16.-, C17.-, C18.-, C19.-, C21.-, C22.-, C23.-, U2.GND, U3.GND, U4.GND
- net IN1_N: now also C12.1; no longer C12.+
- net IN1_P: now also C13.1; no longer C14.+
- net IN2_N: now also C18.1; no longer C17.+
- net IN2_P: now also C19.1; no longer C19.+
- net IN3_N: now also C16.1; no longer C16.+
- net IN3_P: now also C17.1; no longer C18.+
- net IN4_N: now also C22.1; no longer C21.+
- net IN4_P: now also C23.1, R10.2; no longer C23.+, R12.2
- net N$1: now also C10.+, C11.+; no longer C5.+, C6.+
- net N$2: now also C10.-, C11.-; no longer C5.-, C6.-
- net N$3: now also C24.+; no longer C7.+
- net N$4: now also C5.+; no longer C10.+
- net N$5: now also C7.+; no longer C8.+
- net N$6: now also C8.+; no longer C11.+
- net SRB1: no longer U2.IO4
- net SRB2: no longer U2.IO3
- net _SRB1: now also C15.1; no longer C15.+
- net _SRB2: now also C14.1; no longer C13.+
Other:
- moved on the sheet: C10, C11, C5, C7, C8, R10, R12

Commit message: modified:   ADS1299_4_Feather.brd 	modified:   ADS1299_4_Feather.sch
Parts:
- removed C23: 1 nF, adafruit:C-US025-024X044
- removed C7: 100uF, SparkFun-Capacitors:10UF-POLAR-RADIAL-2.5MM-25V-20%
- removed R9: 1M, adafruit:R-US_0207/10
- added C20: 100uF, SparkFun-Capacitors:10UF-0805-10V-10%
- added C25: 1nF, SparkFun-Capacitors:10UF-0805-10V-10%
- added R13: 1M, SparkFun-Resistors:RESISTOR0805
- C1, C10, C2, C24, C3, C4, C5, C8, C9: device SparkFun-Capacitors:10UF-POLAR-RADIAL-2.5MM-25V-20% -> SparkFun-Capacitors:10UF-0805-10V-10%
- C11: value 0.1uF -> 1nF; device SparkFun-Capacitors:10UF-POLAR-RADIAL-2.5MM-25V-20% -> SparkFun-Capacitors:10UF-0805-10V-10%
- C12, C13, C14, C15, C16, C17, C18, C19, C21, C22: value 1 nF -> 1nF; device adafruit:C-US025-024X044 -> SparkFun-Capacitors:10UF-0805-10V-10%
- C6: value 1 nF -> 0.1uF; device adafruit:C-US025-024X044 -> SparkFun-Capacitors:10UF-0805-10V-10%
- FRAME1: REV 1 -> 2
- R1, R10, R11, R12, R2, R3, R4, R5, R6, R7, R8: device SparkFun-Resistors:1MOHM-HORIZ-1/6W-5% -> SparkFun-Resistors:RESISTOR0805
Connections:
- removed net N$2: C10.-, C11.-, U1.RESV1, U1.VREFN
- net 3V3: now also C3.1, C4.1; no longer C3.+, C4.+
- net 4_P: now also R12.1; no longer R10.1
- net 5V: now also C1.1, C2.1; no longer C1.+, C2.+
- net BIAS: now also R10.1; no longer R12.1
- net BIAS_DRV: now also C19.1, C25.1, R10.2, R13.1; no longer C21.1, C6.1, R12.2, R9.2
- net BIAS_IN: now also C25.2, R13.2; no longer C6.2, R9.1
- net GND: now also C1.2, C10.2, C11.2, C2.2, C20.2, C24.2, C3.2, C4.2, C5.2, C6.2, C8.2, C9.2, U1.RESV1, U1.VREFN; no longer C1.-, C2.-, C23.2, C24.-, C3.-, C4.-, C5.-, C7.-, C8.-, C9.-
- net IN1_N: now also C11.1; no longer C12.1
- net IN1_P: now also C12.1; no longer C13.1
- net IN2_N: now also C17.1; no longer C18.1
- net IN2_P: now also C18.1; no longer C19.1
- net IN3_N: now also C15.1; no longer C16.1
- net IN3_P: now also C16.1; no longer C17.1
- net IN4_N: now also C21.1; no longer C22.1
- net IN4_P: now also C22.1, R12.2; no longer C23.1, R10.2
- net N$1: now also C10.1, C5.1; no longer C10.+, C11.+
- net N$3: now also C24.1; no longer C24.+
- net N$4: now also C6.1, C8.1; no longer C5.+, C9.+
- net N$5: now also C20.1; no longer C7.+
- net N$6: now also C9.1; no longer C8.+
- net _SRB1: now also C14.1; no longer C15.1
- net _SRB2: now also C13.1; no longer C14.1
Other:
- moved on the sheet: C12, C13, C14, C15, C16, C17, C18, C19, C21, C22, C6, R10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

Commit message: Increased distance between adafruit mounting headers from 0.7" to 0.8"
	modified:   ADS1299_4_Feather.brd
	modified:   ADS1299_4_Feather.sch
Parts:
- FRAME1: REV 2 -> 3
Changed lines of the file:
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@@
 <part name="FRAME1" library="SparkFun-Aesthetics" deviceset="FRAME-LEDGER" device="">
 <attribute name="DESIGNER" value="Ian Romano"/>
-<attribute name="REV" value="2"/>
+<attribute name="REV" value="3"/>
 </part>
 <part name="C20" library="SparkFun-Capacitors" deviceset="10UF" device="-0805-10V-10%" value="100uF"/>
