File: ADS1299_feather/ADS1299_4_Feather.sch (EAGLE design)
At the start: 40 parts, among them U1 ADS1299-4PAG

Commit message: Uploading final standalone and feather files
Parts:
- removed C11, C12, C13, C14, C15, C16, C17, C18, C19, C21, C22: 1nF, SparkFun-Capacitors:10UF-0805-10V-10%
- removed JP1: 1x12, Proto FeatherWing:MICROBUILDER_HEADER-1X1276MIL
- removed JP2: 1x16, Proto FeatherWing:MICROBUILDER_HEADER-1X16_76MIL
- removed JP3: 2x9, adafruit:PINHD-2X9-BIG
- removed R1, R10, R11, R12, R2, R3, R4, R5, R6, R7, R8: 2.2k, SparkFun-Resistors:RESISTOR0805
- added BOTTOM: (no value), ADS_Feather:MICROBUILDER_HEADER-1X16_76MIL
- added CA1, CA2, CA3, CA4, CA5: 1nF, ADS_Feather:SLEEPSURELIB_W2A45C103MAT2A
- added ELECTRODES: (no value), ADS_Feather:SLEEPSURELIB_PINHD-2X10-BIG
- added RA1, RA2, RA3, RA4, RA5: 2.2k, ADS_Feather:SLEEPSURELIB_EXB-28V222JX
- added TOP: (no value), ADS_Feather:MICROBUILDER_HEADER-1X1276MIL
- added U$1, U$2: MRB120, ADS_Feather:MBR160HW
Connections:
- removed net CLK0: JP1.6, JP1.8, U1.CLK
- removed net EN: JP1.2
- removed net RESET: JP2.1
- new net 5_N: ELECTRODES.N5, RA3.R4B
- new net 5_P: ELECTRODES.P5, RA3.R3B
- new net 6_N: ELECTRODES.N6, RA4.R2B
- new net 6_P: ELECTRODES.P6, RA4.R1B
- new net 7_N: ELECTRODES.N7, RA4.R4B
- new net 7_P: ELECTRODES.P7, RA4.R3B
- new net 8_N: ELECTRODES.N8, RA5.R2B
- new net 8_P: ELECTRODES.P8, RA5.R1B
- new net ADS_START: TOP.27, U1.START
- new net GPIO1: TOP.13, U1.GPIO1
- new net GPIO2: TOP.33, U1.GPIO2
- new net IN5_N: CA3.C1B, RA3.R4A, U1.IN5N
- new net IN5_P: CA3.C2B, RA3.R3A, U1.IN5P
- new net IN6_N: CA4.C3B, RA4.R2A, U1.IN6N
- new net IN6_P: CA4.C4B, RA4.R1A, U1.IN6P
- new net IN7_N: CA4.C1B, RA4.R4A, U1.IN7N
- new net IN7_P: CA4.C2B, RA4.R3A, U1.IN7P
- new net IN8_N: CA5.C3B, RA5.R2A, U1.IN8N
- new net IN8_P: CA5.C4B, RA5.R1A, U1.IN8P
- new net USB: TOP.USB, U$2.A
- net 1_N: now also ELECTRODES.N1, RA1.R4B; no longer JP3.14, R1.1
- net 1_P: now also ELECTRODES.P1, RA1.R3B; no longer JP3.13, R2.1
- net 2_N: now also ELECTRODES.N2, RA2.R2B; no longer JP3.12, R7.1
- net 2_P: now also ELECTRODES.P2, RA2.R1B; no longer JP3.11, R8.1
- net 3V3: now also BOTTOM.3V; no longer JP2.2
- net 3_N: now also ELECTRODES.N3, RA2.R4B; no longer JP3.10, R5.1
- net 3_P: now also ELECTRODES.P3, RA2.R3B; no longer JP3.9, R6.1
- net 4_N: now also ELECTRODES.N4, RA3.R2B; no longer JP3.8, R11.1
- net 4_P: now also ELECTRODES.P4, RA3.R1B; no longer JP3.7, R12.1
- net 5V: now also U$1.C, U$2.C; no longer JP1.3, JP3.1, JP3.2, U1.IN5N, U1.IN5P, U1.IN6N, U1.IN6P, U1.IN7N, U1.IN7P, U1.IN8N, U1.IN8P
- net ADS_RESET: now also TOP.32; no longer JP1.9
- net BATT: now also TOP.BAT, U$1.A; no longer JP1.1
- net BIAS: now also ELECTRODES.BIAS1, ELECTRODES.BIAS2, RA5.R4B; no longer JP3.5, JP3.6, R10.1
- net BIAS_DRV: now also RA5.R4A; no longer C19.1, R10.2
- net CS1: now also TOP.14; no longer JP1.10
- net DRDY: now also TOP.15; no longer JP1.7
- net GND: now also BOTTOM.GND, CA1.C1A, CA1.C2A, CA1.C3A, CA1.C4A, CA2.C1A, CA2.C2A, CA2.C3A, CA2.C4A, CA3.C1A, CA3.C2A, CA3.C3A, CA3.C4A, CA4.C1A, CA4.C2A, CA4.C3A, CA4.C4A, CA5.C1A, CA5.C2A; no longer C11.2, C12.2, C13.2, C14.2, C15.2, C16.2, C17.2, C18.2, C19.2, C21.2, C22.2, JP2.4, JP3.17, JP3.18, JP3.3, JP3.4, U1.GPIO1, U1.GPIO2
- net IN1_N: now also CA1.C1B, RA1.R4A; no longer C11.1, R1.2
- net IN1_P: now also CA1.C2B, RA1.R3A; no longer C12.1, R2.2
- net IN2_N: now also CA2.C3B, RA2.R2A; no longer C17.1, R7.2
- net IN2_P: now also CA2.C4B, RA2.R1A; no longer C18.1, R8.2
- net IN3_N: now also CA2.C1B, RA2.R4A; no longer C15.1, R5.2
- net IN3_P: now also CA2.C2B, RA2.R3A; no longer C16.1, R6.2
- net IN4_N: now also CA3.C3B, RA3.R2A; no longer C21.1, R11.2
- net IN4_P: now also CA3.C4B, RA3.R1A; no longer C22.1, R12.2
- net MISO: now also BOTTOM.MISO; no longer JP2.13
- net MOSI: now also BOTTOM.MOSI; no longer JP2.12
- net SCLK: now also BOTTOM.SCK; no longer JP2.11
- net SRB1: now also ELECTRODES.SRB1, RA1.R2B; no longer JP3.15, R4.1
- net SRB2: now also ELECTRODES.SRB2, RA1.R1B; no longer JP3.16, R3.1
- net _SRB1: now also CA1.C3B, RA1.R2A; no longer C14.1, R4.2
- net _SRB2: now also CA1.C4B, RA1.R1A; no longer C13.1, R3.2
