File: Standalone/SleepSureStandAloneV2.sch (EAGLE design)
At the start: 60 parts, among them IC1 CP2104, Q1 mmbt2222, Q2 mmbt2222, Q3 DMG3415U, SW2 KMR2, U1 ADS1299-4PAG, U2 AP2112-3.3, U3 MCP73831T-2ACI/OT, X1 JSTPH, X2 ESP32_WROOM32_SKINNY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

Commit message: modified design file and removed errors
Parts:
- removed X4: 20329, microbuilder:USB_MICRO_20329_V2
- added C17: 10uF, microbuilder:CAP_CERAMIC0805-NOOUTLINE
- added C18: 2.2uF, microbuilder:CAP_CERAMIC0805-NOOUTLINE
- added C19: 0.1uF, microbuilder:CAP_CERAMIC0805_10MGAP
- added C22: 100uF, SparkFun-Capacitors:10UF-0805-10V-10%
- added J1: 10118192-0002LF, ADS_Feather:10118192-0002LF
- added LED1: RED, microbuilder:LED0805_NOOUTLINE
- added LED2: BLUE, microbuilder:LED0805_NOOUTLINE
- added R11, R9: 1k, SparkFun-Resistors:RESISTOR0805
- added R16: 1.87M, SparkFun-Resistors:RESISTOR0805
- added R17: 340k, SparkFun-Resistors:RESISTOR0805
- added R18: 1.8M, SparkFun-Resistors:RESISTOR0805
- added R19, R5: 200k, SparkFun-Resistors:RESISTOR0805
- added T1: MMUN2133LT1G, transistor:MUN2114T1-PNP_DRIVER-SC59-BEC
- added U$55: 6.8uH, ADS_Feather:ASPI-0628-6R8M-T1
- added U$62, U$66: MRB120, ADS_Feather:MBR160HW
- added U4: TPS61090RSAR, microbuilder:VREG_TPS6103X
- FRAME2: DESIGNER Ian Romano -> Matias Saavedra Silva; DESIGNER2 (none) -> Ian Romano
- U$23, U$46, U$48, U$50, U$52: value W2A45C103MAT2A -> 1nF
- U$44, U$45, U$47, U$49, U$51: value (none) -> 2.2k
Connections:
- removed net IO14_A6: X2.IO14/A2_6
- removed net IO15_A8: X2.IO15/A2_3
- removed net IO32_A7: X2.IO32/A1_4/X32P
- removed net N$2: IC1G$1.D+, X4.D+
- removed net N$6: IC1G$1.D-, X4.D-
- removed net SCLK: U1.SCLK
- new net 5VBAT: C18.1, C22.1, R18.2, R9.2, U$66.A, U4.VOUT
- new net D+: IC1G$1.D+, J1.D+
- new net D-: IC1G$1.D-, J1.D-
- new net ENABLE: R5.1, U4.EN
- new net GPIO0: Q2.C, X2.IO0/A2_1
- new net IO16: X2.IO16
- new net LBO: T1.B, U4.LBO
- new net N$16: U$55.2, U4.SW
- new net N$17: R16.1, R17.2, U4.LBI
- new net N$18: R18.1, R19.2, U4.FB
- new net N$19: LED2.A, R9.1
- new net N$20: LED1.A, R11.1
- new net N$21: R11.2, T1.C
- net 5V: now also U$62.C, U$66.C
- net ADS_CS: now also X2.IO14/A2_6; no longer Q2.C, X2.IO0/A2_1
- net ADS_RESET: now also X2.IO32/A1_4/X32P
- net DRDY: now also X2.IO15/A2_3; no longer X2.IO16
- net GND: now also C17.2, C18.2, C19.2, C22.2, J1.GND, LED1.C, LED2.C, R17.1, R19.1, U4.GND, U4.PGND, U4.SYNC; no longer X4.GND
- net SCK: now also U1.SCLK
- net VBAT: now also C17.1, C19.1, R16.2, R5.2, T1.E, U$55.1, U4.VBAT
- net VBUS: now also J1.VCC, U$62.A; no longer X4.VBUS
Other:
- note added: "6.8uH power w/2A current"
- note added: "On/Off Switch"
- note added: "See Pg 15 1st para"

Commit message: changed footprint of 100uF caps to 1206
Parts:
- removed C20: 100uF, SparkFun-Capacitors:10UF-0805-10V-10%
- removed U$35: FIDUCIAL_1MM, microbuilder:FIDUCIAL_1MM
- added C21: 0.1uF, SparkFun-Capacitors:10UF-0805-10V-10%
- C19: value 0.1uF -> 100uF; device microbuilder:CAP_CERAMIC0805_10MGAP -> SparkFun-Capacitors:10UF-1206-6.3V-20%
- C22: device SparkFun-Capacitors:10UF-0805-10V-10% -> SparkFun-Capacitors:10UF-1206-6.3V-20%
Connections:
- net 5VBAT: now also C19.1; no longer C22.1
- net GND: now also C21.2; no longer C20.2
- net N$9: now also C22.1; no longer C20.1
- net VBAT: now also C21.1; no longer C19.1
Other:
- moved on the sheet: C19, C22
Changed lines of the file:
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@@
 <part name="U$30" library="microbuilder" deviceset="GND" device=""/>
 <part name="U$34" library="microbuilder" deviceset="FIDUCIAL" device="_1MM"/>
-<part name="U$35" library="microbuilder" deviceset="FIDUCIAL" device="_1MM"/>
 <part name="U$31" library="microbuilder" deviceset="MOUNTINGHOLE" device="2.5"/>
 <part name="U$32" library="microbuilder" deviceset="MOUNTINGHOLE" device="2.5"/>
@@
 <attribute name="REV" value="2"/>
 </part>
-<part name="C20" library="SparkFun-Capacitors" deviceset="10UF" device="-0805-10V-10%" value="100uF"/>
 <part name="C10" library="SparkFun-Capacitors" deviceset="10UF" device="-0805-10V-10%" value="10uF"/>
 <part name="C5" library="SparkFun-Capacitors" deviceset="10UF" device="-0805-10V-10%" value="1uF"/>
@@
 <part name="U$57" library="microbuilder" deviceset="VBAT" device=""/>
 <part name="U$58" library="microbuilder" deviceset="GND" device=""/>
-<part name="C19" library="microbuilder" deviceset="CAP_CERAMIC" device="0805_10MGAP" value="0.1uF"/>
 <part name="U$59" library="microbuilder" deviceset="GND" device=""/>
 <part name="U$60" library="microbuilder" deviceset="GND" device=""/>
@@
 <part name="R9" library="SparkFun-Resistors" deviceset="RESISTOR" device="0805" value="1k"/>
 <part name="R11" library="SparkFun-Resistors" deviceset="RESISTOR" device="0805" value="1k"/>
-<part name="C22" library="SparkFun-Capacitors" deviceset="10UF" device="-0805-10V-10%" value="100uF"/>
 <part name="U$55" library="ADS_Feather" deviceset="ASPI-0628-6R8M-T1" device="" value="6.8uH"/>
 <part name="R5" library="SparkFun-Resistors" deviceset="RESISTOR" device="0805" value="200k"/>
@@
 <part name="U$66" library="ADS_Feather" deviceset="MBR160HW" device="" value="MRB120"/>
 <part name="J1" library="ADS_Feather" deviceset="10118192-0002LF" device=""/>
+<part name="C21" library="SparkFun-Capacitors" deviceset="10UF" device="-0805-10V-10%" value="0.1uF"/>
+<part name="C19" library="SparkFun-Capacitors" library_urn="urn:adsk.eagle:library:510" deviceset="10UF" device="-1206-6.3V-20%" package3d_urn="urn:adsk.eagle:package:37426/1" value="100uF"/>
+<part name="C22" library="SparkFun-Capacitors" library_urn="urn:adsk.eagle:library:510" deviceset="10UF" device="-1206-6.3V-20%" package3d_urn="urn:adsk.eagle:package:37426/1" value="100uF"/>
 </parts>
 <sheets>
@@
 </instance>
 <instance part="U$34" gate="G$1" x="231.14" y="25.4" smashed="yes"/>
-<instance part="U$35" gate="G$1" x="228.6" y="25.4" smashed="yes"/>
 <instance part="U$31" gate="G$1" x="236.22" y="25.4" smashed="yes"/>
 <instance part="U$32" gate="G$1" x="241.3" y="25.4" smashed="yes"/>
@@
 <attribute name="REV" x="-20.32" y="6.604" size="2.7432" layer="94" font="vector"/>
 <attribute name="DESIGNER2" x="-86.36" y="7.62" size="2.7432" layer="94" font="vector"/>
-</instance>
-<instance part="C20" gate="G$1" x="-256.54" y="15.24" smashed="yes">
-<attribute name="NAME" x="-255.016" y="18.161" size="1.778" layer="95" font="vector"/>
-<attribute name="VALUE" x="-255.016" y="13.081" size="1.778" layer="96" font="vector"/>
 </instance>
 <instance part="C10" gate="G$1" x="-381" y="38.1" smashed="yes">
@@
 <attribute name="VALUE" x="-174.244" y="140.716" size="1.27" layer="96"/>
 </instance>
-<instance part="U$58" gate="G$1" x="-193.04" y="81.28" smashed="yes">
-<attribute name="VALUE" x="-194.564" y="78.74" size="1.27" layer="96"/>
-</instance>
-<instance part="C19" gate="G$1" x="-193.04" y="86.36" smashed="yes">
-<attribute name="NAME" x="-195.33" y="87.61" size="1.27" layer="95" font="vector" rot="R90" align="center"/>
-<attribute name="VALUE" x="-190.74" y="87.61" size="1.27" layer="96" font="vector" rot="R90" align="center"/>
+<instance part="U$58" gate="G$1" x="-193.04" y="78.74" smashed="yes">
+<attribute name="VALUE" x="-194.564" y="76.2" size="1.27" layer="96"/>
 </instance>
 <instance part="U$59" gate="G$1" x="-129.54" y="55.88" smashed="yes">
@@
 <attribute name="VALUE" x="-112.776" y="66.04" size="1.778" layer="96" font="vector" rot="R90" align="top-center"/>
 </instance>
-<instance part="C22" gate="G$1" x="-127" y="93.98" smashed="yes">
-<attribute name="NAME" x="-125.476" y="96.901" size="1.778" layer="95" font="vector"/>
-<attribute name="VALUE" x="-125.476" y="91.821" size="1.778" layer="96" font="vector"/>
-</instance>
 <instance part="U$55" gate="G$1" x="-185.42" y="99.06" smashed="yes" rot="R90">
 <attribute name="NAME" x="-191.77" y="101.6" size="1.778" layer="95" rot="R90"/>
@@
 <attribute name="NAME" x="160.02" y="133.35" size="1.778" layer="95" rot="MR0"/>
 <attribute name="VALUE" x="162.56" y="109.22" size="1.778" layer="96" rot="MR0"/>
+</instance>
+<instance part="C21" gate="G$1" x="-193.04" y="86.36" smashed="yes">
+<attribute name="NAME" x="-191.516" y="89.281" size="1.778" layer="95" font="vector"/>
+<attribute name="VALUE" x="-191.516" y="84.201" size="1.778" layer="96" font="vector"/>
+</instance>
+<instance part="C19" gate="G$1" x="-127" y="93.98" smashed="yes">
+<attribute name="NAME" x="-125.476" y="96.901" size="1.778" layer="95" font="vector"/>
+<attribute name="VALUE" x="-125.476" y="91.821" size="1.778" layer="96" font="vector"/>
+</instance>
+<instance part="C22" gate="G$1" x="-256.54" y="15.24" smashed="yes">
+<attribute name="NAME" x="-255.016" y="18.161" size="1.778" layer="95" font="vector"/>
+<attribute name="VALUE" x="-255.016" y="13.081" size="1.778" layer="96" font="vector"/>
 </instance>
 </instances>
@@
 <junction x="-256.54" y="5.08"/>
 <pinref part="C24" gate="G$1" pin="2"/>
-<pinref part="C20" gate="G$1" pin="2"/>
+<pinref part="C22" gate="G$1" pin="2"/>
 </segment>
 <segment>
@@
 </segment>
 <segment>
-<pinref part="C19" gate="G$1" pin="2"/>
-<pinref part="U$58" gate="G$1" pin="GND"/>
-</segment>
-<segment>
 <wire x1="-142.24" y1="78.74" x2="-137.16" y2="78.74" width="0.1524" layer="91"/>
 <pinref part="U4" gate="G$1" pin="PGND"/>
@@
 <wire x1="-127" y1="88.9" x2="-124.46" y2="88.9" width="0.1524" layer="91"/>
 <pinref part="U$61" gate="G$1" pin="GND"/>
-<pinref part="C22" gate="G$1" pin="2"/>
+<pinref part="C19" gate="G$1" pin="2"/>
 </segment>
 <segment>
@@
 <wire x1="165.1" y1="119.38" x2="170.18" y2="119.38" width="0.1524" layer="91"/>
 <wire x1="170.18" y1="119.38" x2="170.18" y2="114.3" width="0.1524" layer="91"/>
+</segment>
+<segment>
+<pinref part="U$58" gate="G$1" pin="GND"/>
+<pinref part="C21" gate="G$1" pin="2"/>
+<wire x1="-193.04" y1="81.28" x2="-193.04" y2="83.82" width="0.1524" layer="91"/>
 </segment>
 </net>
@@
 <pinref part="C17" gate="G$1" pin="1"/>
 <pinref part="U$56" gate="G$1" pin="VBAT"/>
-<pinref part="C19" gate="G$1" pin="1"/>
 <pinref part="R16" gate="G$1" pin="2"/>
 <junction x="-185.42" y="93.98"/>
@@
 <junction x="-200.66" y="99.06"/>
 <pinref part="U$55" gate="G$1" pin="1"/>
+<pinref part="C21" gate="G$1" pin="1"/>
 </segment>
 <segment>
@@
 <wire x1="-304.8" y1="25.4" x2="-256.54" y2="25.4" width="0.1524" layer="91"/>
 <wire x1="-256.54" y1="25.4" x2="-256.54" y2="20.32" width="0.1524" layer="91"/>
-<pinref part="C20" gate="G$1" pin="1"/>
+<pinref part="C22" gate="G$1" pin="1"/>
 </segment>
 </net>
@@
 <wire x1="-132.08" y1="99.06" x2="-132.08" y2="96.52" width="0.1524" layer="91"/>
 <junction x="-137.16" y="99.06"/>
-<pinref part="C22" gate="G$1" pin="1"/>
+<junction x="-132.08" y="99.06"/>
 <wire x1="-132.08" y1="99.06" x2="-127" y2="99.06" width="0.1524" layer="91"/>
-<junction x="-132.08" y="99.06"/>
+<pinref part="R9" gate="G$1" pin="2"/>
 <wire x1="-127" y1="99.06" x2="-114.3" y2="99.06" width="0.1524" layer="91"/>
-<junction x="-127" y="99.06"/>
-<pinref part="R9" gate="G$1" pin="2"/>
 <wire x1="-114.3" y1="114.3" x2="-111.76" y2="114.3" width="0.1524" layer="91"/>
 <wire x1="-114.3" y1="99.06" x2="-114.3" y2="114.3" width="0.1524" layer="91"/>
 <label x="-114.3" y="99.06" size="1.778" layer="95"/>
-</segment>
-<segment>
+<pinref part="C19" gate="G$1" pin="1"/>
+<junction x="-127" y="99.06"/>
+</segment>
+<segment>

Commit message: added START pin of ADS1299 to gpio27
Connections:
- removed net IO27_A10: X2.IO27/A2_7
- new net ADS_START: U1.START, X2.IO27/A2_7
Changed lines of the file:
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@@
-</segment>
-</net>
-<net name="IO27_A10" class="0">
-<segment>
-<wire x1="78.74" y1="73.66" x2="91.44" y2="73.66" width="0.1524" layer="91"/>
-<label x="81.28" y="73.66" size="1.778" layer="95"/>
-<pinref part="X2" gate="G$1" pin="IO27/A2_7"/>
 </segment>
 </net>
@@
 </segment>
 </net>
+<net name="ADS_START" class="0">
+<segment>
+<pinref part="U1" gate="G$1" pin="START"/>
+<wire x1="-340.36" y1="50.8" x2="-365.76" y2="50.8" width="0.1524" layer="91"/>
+<label x="-365.76" y="50.8" size="1.778" layer="95"/>
+</segment>
+<segment>
+<wire x1="78.74" y1="73.66" x2="91.44" y2="73.66" width="0.1524" layer="91"/>
+<label x="81.28" y="73.66" size="1.778" layer="95"/>
+<pinref part="X2" gate="G$1" pin="IO27/A2_7"/>
+</segment>
+</net>

Commit message: Uploading final standalone and feather files
Parts:
- removed R13: 10K, microbuilder:RESISTOR_4PACK
- removed U$34: FIDUCIAL_1MM, microbuilder:FIDUCIAL_1MM
- added U$7: 10k, SleepSureLib:EXB-28V222JX
- FRAME2: DESIGNER Matias Saavedra Silva -> Ian Romano; DESIGNER2 Ian Romano -> Matias Saavedra Silva; REV 2 -> 3
- JP2: value (none) -> 2x10
- U3: value MCP73831T-2ACI/OT -> LiPoly
- renumbered X1 to 2PIN
Connections:
- removed net N$12: Q1.B, R13G$4.2
- removed net N$13: Q2.B, R13G$2.1
- new net N$2: Q2.B, U$7.P$5
- new net N$6: Q1.B, U$7.P$4
- net 3.3V: now also U$7.P$6; no longer R13G$3.1
- net DTR: now also U$7.P$8; no longer R13G$4.1
- net RESET: now also U$7.P$2; no longer R13G$3.2
- net RTS: now also U$7.P$1; no longer R13G$2.2
Other:
- moved on the sheet: Q1, Q2, R1, R3
